Commit message: 版本大更新
1. 手部映射关节角传输tcp->ros2
2. 模型更改
2. 图像获取改为realsense

File: assets/inspire_hand/inspire_hand_left.urdf (robot description, URDF)
Before this commit: robot h1, 18 links, 17 joints
Links:
- removed link L_hand_base_link
- removed link L_index_intermediate
- removed link L_index_proximal
- removed link L_index_tip
- removed link L_middle_intermediate
- removed link L_middle_proximal
- removed link L_middle_tip
- removed link L_pinky_intermediate
- removed link L_pinky_proximal
- removed link L_pinky_tip
- removed link L_ring_intermediate
- removed link L_ring_proximal
- removed link L_ring_tip
- removed link L_thumb_distal
- removed link L_thumb_intermediate
- removed link L_thumb_proximal
- removed link L_thumb_proximal_base
- removed link L_thumb_tip
- added link base
- added link hand_base_link, mass 0.14143; collision box size=0.0125 0.0111 0.0089; collision box size=0.0125 0.0111 0.0089
- added link index_intermediate, mass 0.0045683; collision mesh filename=meshes/collision/left_index_intermediate.obj; visual mesh filename=meshes/visual/left_index_intermediate.glb
- added link index_proximal, mass 0.0042403; collision mesh filename=meshes/collision/left_index_proximal.obj; visual mesh filename=meshes/visual/left_index_proximal.glb
- added link index_tip
- added link middle_intermediate, mass 0.0050396; collision mesh filename=meshes/collision/left_middle_intermediate.obj; visual mesh filename=meshes/visual/left_middle_intermediate.glb
- added link middle_proximal, mass 0.0042403; collision mesh filename=meshes/collision/left_index_proximal.obj; visual mesh filename=meshes/visual/left_index_proximal.glb
- added link middle_tip
- added link pinky_intermediate, mass 0.0035996; collision mesh filename=meshes/collision/left_pinky_intermediate.obj; visual mesh filename=meshes/visual/left_pinky_intermediate.glb
- added link pinky_proximal, mass 0.0042403; collision mesh filename=meshes/collision/left_index_proximal.obj; visual mesh filename=meshes/visual/left_index_proximal.glb
- added link pinky_tip
- added link ring_intermediate, mass 0.0045683; collision mesh filename=meshes/collision/left_index_intermediate.obj; visual mesh filename=meshes/visual/left_index_intermediate.glb
- added link ring_proximal, mass 0.0042403; collision mesh filename=meshes/collision/left_index_proximal.obj; visual mesh filename=meshes/visual/left_index_proximal.glb
- added link ring_tip
- added link thumb_distal, mass 0.0033441; collision mesh filename=meshes/collision/left_thumb_distal.obj scale=1 1 1; visual mesh filename=meshes/visual/left_thumb_distal.glb
- added link thumb_intermediate, mass 0.0037847; collision mesh filename=meshes/collision/left_thumb_intermediate.obj; visual mesh filename=meshes/visual/left_thumb_intermediate.glb
- added link thumb_proximal, mass 0.0066075; collision mesh filename=meshes/collision/left_thumb_proximal.obj; visual mesh filename=meshes/visual/left_thumb_proximal.glb
- added link thumb_proximal_base, mass 0.0018869; collision mesh filename=meshes/collision/left_thumb_proximal_base.obj; visual mesh filename=meshes/visual/left_thumb_proximal_base.glb
- added link thumb_tip
Joints:
- removed joint L_index_intermediate_joint
- removed joint L_index_proximal_joint
- removed joint L_index_tip_joint
- removed joint L_middle_intermediate_joint
- removed joint L_middle_proximal_joint
- removed joint L_middle_tip_joint
- removed joint L_pinky_intermediate_joint
- removed joint L_pinky_proximal_joint
- removed joint L_pinky_tip_joint
- removed joint L_ring_intermediate_joint
- removed joint L_ring_proximal_joint
- removed joint L_ring_tip_joint
- removed joint L_thumb_distal_joint
- removed joint L_thumb_intermediate_joint
- removed joint L_thumb_proximal_pitch_joint
- removed joint L_thumb_proximal_yaw_joint
- removed joint L_thumb_tip_joint
- added joint base_joint: type fixed, parent base, child hand_base_link, origin xyz=0 0 0 rpy=0 0 0
- added joint index_intermediate_joint: type revolute, parent index_proximal, child index_intermediate, origin xyz=-0.0026138 -0.032026 -0.001 rpy=0 0 0, axis 0 0 -1, limit lower=-0.04545 upper=1.56 effort=1 velocity=0.5, mimic joint=index_proximal_joint multiplier=1.06399 offset=-0.04545
- added joint index_proximal_joint: type revolute, parent hand_base_link, child index_proximal, origin xyz=0.00028533 -0.13653 0.032268 rpy=-0.034907 0 0, axis 0 0 -1, limit lower=0 upper=1.47 effort=1 velocity=0.5
- added joint index_tip_joint: type fixed, parent index_intermediate, child index_tip, origin xyz=-0.0008 -0.045 -0.005 rpy=0 0 0
- added joint middle_intermediate_joint: type revolute, parent middle_proximal, child middle_intermediate, origin xyz=-0.0024229 -0.032041 -0.001 rpy=0 0 0, axis 0 0 -1, limit lower=-0.04545 upper=1.56 effort=1 velocity=0.5, mimic joint=middle_proximal_joint multiplier=1.06399 offset=-0.04545
- added joint middle_proximal_joint: type revolute, parent hand_base_link, child middle_proximal, origin xyz=0.00028533 -0.1371 0.01295 rpy=0 0 0, axis 0 0 -1, limit lower=0 upper=1.47 effort=1 velocity=0.5
- added joint middle_tip_joint: type fixed, parent middle_intermediate, child middle_tip, origin xyz=-0.001 -0.048 -0.005 rpy=0 0 0
- added joint pinky_intermediate_joint: type revolute, parent pinky_proximal, child pinky_intermediate, origin xyz=-0.0024229 -0.032041 -0.001 rpy=0 0 0, axis 0 0 -1, limit lower=-0.04545 upper=1.56 effort=1 velocity=0.5, mimic joint=pinky_proximal_joint multiplier=1.06399 offset=-0.04545
- added joint pinky_proximal_joint: type revolute, parent hand_base_link, child pinky_proximal, origin xyz=0.00028533 -0.13571 -0.025488 rpy=0.10472 0 0, axis 0 0 -1, limit lower=0 upper=1.47 effort=1 velocity=0.5
- added joint pinky_tip_joint: type fixed, parent pinky_intermediate, child pinky_tip, origin xyz=-0.0008 -0.037 -0.005 rpy=0 0 0
- added joint ring_intermediate_joint: type revolute, parent ring_proximal, child ring_intermediate, origin xyz=-0.0024229 -0.032041 -0.001 rpy=0 0 0, axis 0 0 -1, limit lower=-0.04545 upper=1.56 effort=1 velocity=0.5, mimic joint=ring_proximal_joint multiplier=1.06399 offset=-0.04545
- added joint ring_proximal_joint: type revolute, parent hand_base_link, child ring_proximal, origin xyz=0.00028533 -0.13691 -0.0062872 rpy=0.05236 0 0, axis 0 0 -1, limit lower=0 upper=1.47 effort=1 velocity=0.5
- added joint ring_tip_joint: type fixed, parent ring_intermediate, child ring_tip, origin xyz=-0.0008 -0.045 -0.005 rpy=0 0 0
- added joint thumb_distal_joint: type revolute, parent thumb_intermediate, child thumb_distal, origin xyz=0.020248 -0.010156 -0.0012 rpy=0 0 0, axis 0 0 -1, limit lower=0 upper=0.4 effort=1 velocity=0.5, mimic joint=thumb_proximal_pitch_joint multiplier=0.667 offset=0
- added joint thumb_intermediate_joint: type revolute, parent thumb_proximal, child thumb_intermediate, origin xyz=0.04407 -0.034553 -0.0008 rpy=0 0 0, axis 0 0 -1, limit lower=0 upper=0.8 effort=1 velocity=0.5, mimic joint=thumb_proximal_pitch_joint multiplier=1.334 offset=0
- added joint thumb_proximal_pitch_joint: type revolute, parent thumb_proximal_base, child thumb_proximal, origin xyz=0.0099867 0.0098242 -0.0089 rpy=-1.5708 0 0.16939, axis 0 0 -1, limit lower=0 upper=0.6 effort=1 velocity=0.5
- added joint thumb_proximal_yaw_joint: type revolute, parent hand_base_link, child thumb_proximal_base, origin xyz=-0.01696 -0.0691 0.02045 rpy=1.5708 -1.5708 0, axis 0 0 1, limit lower=0 upper=1.308 effort=1 velocity=0.5
- added joint thumb_tip_joint: type fixed, parent thumb_distal, child thumb_tip, origin xyz=0.0202 -0.0140 -0.006 rpy=0 0 0

File: assets/inspire_hand/inspire_hand_right_glb.urdf (robot description, URDF)
Before this commit: robot inspire_hand_right, 19 links, 18 joints
Joints:
- joint base_joint: origin xyz=0 0 0 rpy=0 0 0 -> xyz=0 0 0 rpy=-1.57079 0 3.14159
